Commit message: buat package comm

File: src/urdf_raditya/urdf/urdf_raditya.urdf (robot description, URDF)
Before this commit: robot urdf_raditya, 9 links, 8 joints
Links:
- removed link enpoint1
- removed link enpoint2
- removed link motor1 
- removed link motor4_1 
- added link motor1, mass 0.0545469130635853; collision mesh filename=package://urdf_raditya/meshes/motor1.STL; visual mesh filename=package://urdf_raditya/meshes/motor1.STL
- added link motor4_1, mass 0.0077585; collision mesh filename=package://urdf_raditya/meshes/motor4_1.STL; visual mesh filename=package://urdf_raditya/meshes/motor4_1.STL
Joints:
- removed joint enpoint1
- removed joint enpoint2
- joint motor4_1: child motor4_1  -> motor4_1
- joint servomotor1: child motor1  -> motor1
- joint servomotor2: parent motor1  -> motor1
