Commit message: urdf sudah benar

File: src/urdffp/urdf/urdffp.urdf (robot description, URDF)
Before this commit: robot URDFFPRADITYA, 9 links, 8 joints
Links:
- removed link endpoint1
- removed link endpoint2
- removed link servo4
- removed link servolink1
- removed link servolink2
- removed link servolink3
- removed link servotipu
- added link endpointgear, mass 0.605238076529163; collision mesh filename=package://urdffp/meshes/endpointgear.STL; visual mesh filename=package://urdffp/meshes/endpointgear.STL
- added link endpointpalsu, mass 0.605238076529163; collision mesh filename=package://urdffp/meshes/endpointpalsu.STL; visual mesh filename=package://urdffp/meshes/endpointpalsu.STL
- added link link1, mass 0.0802065215999488; collision mesh filename=package://urdffp/meshes/link1.STL; visual mesh filename=package://urdffp/meshes/link1.STL
- added link link2, mass 0.12585545698654; collision mesh filename=package://urdffp/meshes/link2.STL; visual mesh filename=package://urdffp/meshes/link2.STL
- added link link3, mass 0.0260593092533598; collision mesh filename=package://urdffp/meshes/link3.STL; visual mesh filename=package://urdffp/meshes/link3.STL
- added link linkgear1, mass 0.00474004808682916; collision mesh filename=package://urdffp/meshes/linkgear1.STL; visual mesh filename=package://urdffp/meshes/linkgear1.STL
- added link linkgearpalsu, mass 0.00723714741075858; collision mesh filename=package://urdffp/meshes/linkgearpalsu.STL; visual mesh filename=package://urdffp/meshes/linkgearpalsu.STL
- link base: mass 0.272903163990243 -> 0.272903164017977; geometry collision mesh filename=package://urdffp/meshes/base.STL; visual mesh filename=package://urdffp/meshes/base.STL
- link piringan: mass 0.0882364212328449 -> 0.0882364212464755; geometry collision mesh filename=package://urdffp/meshes/piringan.STL; visual mesh filename=package://urdffp/meshes/piringan.STL
Joints:
- removed joint piringan
- removed joint servo2
- removed joint servo3
- removed joint servo4
- removed joint servotipu
- removed joint sevo1
- added joint servogear: type revolute, parent link3, child linkgear1, origin xyz=0.08705 0.011 -0.0255 rpy=-1.5708 0 0, axis 0 0 1, limit lower=-3.14 upper=3.14 effort=0.17652 velocity=10.472
- added joint servogearpalsu: type revolute, parent link3, child linkgearpalsu, origin xyz=0.08695 0.011 0.0045 rpy=-1.5708 0 0, axis 0 0 1, limit lower=-3.14 upper=3.14 effort=0.17652 velocity=10.472
- added joint servolink1: type revolute, parent piringan, child link1, origin xyz=0.0001138 0 0.054433 rpy=-1.5708 0 0, axis 0 0 -1, limit lower=-3.14 upper=3.14 effort=0.83357 velocity=5.236
- added joint servolink2: type revolute, parent link1, child link2, origin xyz=0.116 0.00030718 0 rpy=0 0 0, axis 0 0 -1, limit lower=-3.14 upper=3.14 effort=0.83357 velocity=5.236
- added joint servolink3: type revolute, parent link2, child link3, origin xyz=0.094648 0.00060842 0 rpy=0 0 0, axis 0 0 1, limit lower=-3.14 upper=3.14 effort=0.83357 velocity=5.236
- added joint servopiringan: type revolute, parent base, child piringan, origin xyz=-3.0958E-05 0 0.0689 rpy=0 0 0, axis -0.0020906 0 -1, limit lower=-3.14 upper=3.14 effort=0.83357 velocity=5.236
- joint endpoint1: child endpoint1 -> endpointgear; origin xyz=0.07851 -0.017246 -0.15499 rpy=0 0 0 -> xyz=0.080522 -0.017346 0 rpy=0 0 0; parent servo4 -> linkgear1
- joint endpoint2: child endpoint2 -> endpointpalsu; origin xyz=0.0762870841043169 0.0128156153922516 -0.154987060760109 rpy=0 0 0 -> xyz=0.080028 0.015057 0 rpy=0 0 0; parent servotipu -> linkgearpalsu

Commit message: progress dikit lah mayan

File: src/urdffp/urdf/urdffp.urdf (robot description, URDF)
Before this commit: robot urdffp, 9 links, 8 joints
Joints:
- joint servolink1: origin xyz=0.0001138 0 0.054433 rpy=-1.5708 0 0 -> xyz=0.0001138 0 0.054433 rpy=-1.5708 -1.5708 0
